Commit message: destroyed seven dof arm to test 5 dof

File: koko_descriptions/koko_description_sevendof_dyn/robots/koko_description_sevendof_dyn.urdf (robot description, URDF)
Before this commit: robot koko_description_sevendof_dyn, 8 links, 7 joints
Links:
- removed link wrist_lift_link
- removed link wrist_roll_link
Joints:
- removed joint wrist_lift_joint
- removed joint wrist_roll_joint

File: koko_descriptions/koko_description_sevendof_kin/robots/koko_description_sevendof_kin.urdf (robot description, URDF)
Before this commit: robot koko_description_sevendof_kin, 12 links, 11 joints
Links:
- removed link ee_tracker_link
- removed link forearm_tracker_link
- removed link wrist_lift_link
- removed link wrist_roll_link
Joints:
- removed joint ee_tracker_joint
- removed joint forearm_tracker_joint
- removed joint wrist_lift_joint
- removed joint wrist_roll_joint
